File: timelapse/2019-07-02_13:30:37_fpga_hat.kicad_pcb (KiCad board)
At the start: 4 copper layers, 65 x 56.5 mm, 90 parts, among them J1 2x20, J2 AudioJack3, J3 Conn_02x06_Top_Bottom, J4 Conn_02x06_Top_Bottom, J5 Conn_02x06_Top_Bottom, J6 Conn_01x02, SW1 PTS815, SW2 PTS815, SW3 PTS815, SW4 PTS815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

Commit message: All parts on board
Parts:
- C1, C11, C2, C26, C27, C3, C4, C5, C6, C7, C8, C9, R1, R2: moved to F.Cu
- moved C28 93.4 mm to (181.4, 50.8)
- moved C13 79.6 mm to (183.7, 53.0), turned to 0 degrees
- moved C23 72.7 mm to (171.4, 59.9)
- moved C6 68.8 mm to (182.2, 55.0)
- moved C14 68.1 mm to (175.9, 55.4), turned to 0 degrees
- moved TP3 66.4 mm to (174.7, 57.5), turned to 0 degrees
- moved C4 65.8 mm to (143.9, 45.1)
- moved C5 64.8 mm to (177.8, 59.1)
- moved C24 64.8 mm to (133.0, 60.7)
- moved R1 64.5 mm to (112.1, 50.5)
- moved C26 61.8 mm to (179.3, 57.1), turned to 0 degrees
- moved U5 60.8 mm to (144.7, 50.3)
- moved C27 60.5 mm to (179.3, 55.1), turned to 0 degrees
- moved C9 57.8 mm to (170.9, 66.1), turned to 0 degrees
- moved C15 57.0 mm to (165.9, 69.8)
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Routing:
- net GND: track 9.05 -> 0.00 mm, vias 4 -> 0
- net +3V3: track 2.83 -> 0.00 mm, vias 5 -> 0
- net +1V2: track 2.26 -> 0.00 mm, vias 4 -> 0
- removed copper zone on In2.Cu, net +3V3
- removed copper zone on In2.Cu, net +5V
