File: timelapse/2019-07-02_20:01:46_fpga_hat.kicad_pcb (KiCad board)
At the start: 4 copper layers, 65 x 56.5 mm, 90 parts, among them J1 2x20, J2 AudioJack3, J3 Conn_02x06_Top_Bottom, J4 Conn_02x06_Top_Bottom, J5 Conn_02x06_Top_Bottom, J6 Conn_01x02, SW1 PTS815, SW2 PTS815, SW3 PTS815, SW4 PTS815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

Commit message: SRAM escaped. Some work on FPGA power routing. Some SRAM pinswapping.
Parts:
- moved R2 3.36 mm to (133.2, 102.6), turned to 90 degrees
- moved C2 2.40 mm to (134.5, 102.5), turned to 90 degrees
Connections:
- U1 pad C4: /SRAM_A11 -> /SRAM_DQ5
- U1 pad J2: /SRAM_A3 -> /SRAM_A16
- U1 pad J5: /SRAM_DQ5 -> /SRAM_A11
- U1 pad K5: /SRAM_A16 -> /SRAM_A3
Routing:
- net /SRAM_A3: track 9.74 -> 21.3 mm
- net /SRAM_A16: track 20.8 -> 9.41 mm
- net GND: track 24.9 -> 14.2 mm, vias 11 -> 7
- net /SRAM_DQ5: track 20.5 -> 10.7 mm
- net /IO1_7: track 9.02 -> 16.7 mm
- net /SRAM_A11: track 11.6 -> 18.1 mm
- net /IO2_3: track 7.98 -> 13.3 mm
- net +1V2: track 12.7 -> 7.71 mm
- net Net-(C2-Pad1): track 4.61 -> 0.00 mm, vias 1 -> 0
- net +3V3: track 10.9 -> 6.70 mm, vias 8 -> 7
- net Net-(C4-Pad1): track 2.83 -> 0.00 mm, vias 1 -> 0
- net Net-(C2-Pad2): track 2.05 -> 0.00 mm, vias 1 -> 0
- net /SRAM_DQ4: track 22.5 -> 20.7 mm
- net /SRAM_A8: track 6.93 -> 8.43 mm
- net Net-(C4-Pad2): track 1.40 -> 0.00 mm, vias 1 -> 0
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