File: timelapse/2019-07-02_20:54:50_fpga_hat.kicad_pcb (KiCad board)
At the start: 4 copper layers, 65 x 56.5 mm, 90 parts, among them J1 2x20, J2 AudioJack3, J3 Conn_02x06_Top_Bottom, J4 Conn_02x06_Top_Bottom, J5 Conn_02x06_Top_Bottom, J6 Conn_01x02, SW1 PTS815, SW2 PTS815, SW3 PTS815, SW4 PTS815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

Commit message: More FPGA escape
Routing:
- net /SRAM_A11: track 16.8 -> 11.6 mm
- net /SRAM_A8: track 10.7 -> 6.93 mm
- net /IO1_7: track 6.90 -> 9.02 mm
- net /SRAM_A16: track 21.7 -> 20.8 mm
- net +3V3: track 13.9 -> 13.1 mm, vias 9 -> 8
- net /IO2_3: track 7.46 -> 7.98 mm
