File: timelapse/2019-07-03_06:45:34_fpga_hat.kicad_pcb (KiCad board)
At the start: 4 copper layers, 65 x 56.5 mm, 90 parts, among them J1 2x20, J2 AudioJack3, J3 Conn_02x06_Top_Bottom, J4 Conn_02x06_Top_Bottom, J5 Conn_02x06_Top_Bottom, J6 Conn_01x02, SW1 PTS815, SW2 PTS815, SW3 PTS815, SW4 PTS815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

Commit message: Continue BGA route-out. SRAM connected, start heading out toward LEDs and IO.
Connections:
- U1 pad A11: /IO0_6 -> /IO0_0
- U1 pad A4: /SW2 -> /IO1_6
- U1 pad A5: /SW1 -> /IO1_4
- U1 pad A6: /LED0 -> /IO1_3
- U1 pad A7: /IO0_4 -> /IO1_2
- U1 pad B4: /LED3 -> /IO2_0
- U1 pad B5: /LED2 -> /IO1_5
- U1 pad B6: /SW0 -> /IO2_6
- U1 pad B7: /AUDIO_L_PWM -> /IO2_5
- U1 pad B8: /IO1_2 -> /IO0_4
- U1 pad C4: /SW3 -> /IO2_1
- U1 pad C7: /AUDIO_R_PWM -> /IO1_1
- U1 pad C8: /IO0_0 -> /IO0_6
- U1 pad D7: /LED1 -> /IO0_7
- U1 pad E8: /IO2_1 -> /SW3
- U1 pad E9: /IO1_6 -> /SW2
- U1 pad F10: /IO2_6 -> /SW0
- U1 pad F11: /IO2_5 -> /AUDIO_L_PWM
- U1 pad F9: /IO1_4 -> /SW1
- U1 pad G8: /IO2_0 -> /LED3
- U1 pad H10: /IO0_7 -> /LED1
- U1 pad J10: /IO1_5 -> /LED2
- U1 pad J8: /GP27_SDIO_DAT3 -> /GP22_SDIO_CLK
- U1 pad K11: /IO1_3 -> /LED0
- U1 pad K6: /GP22_SDIO_CLK -> /GP27_SDIO_DAT3
- U1 pad K7: /IO1_1 -> /AUDIO_R_PWM
Routing:
- net /AUDIO_R_PWM: track 39.3 -> 2.04 mm
- net /IO1_1: track 2.04 -> 38.9 mm
- net /AUDIO_L_PWM: track 36.5 -> 5.10 mm
- net /SW3: track 37.4 -> 8.55 mm
- net /SW0: track 34.7 -> 6.19 mm
- net /SW2: track 33.4 -> 7.96 mm
- net /SW1: track 32.3 -> 6.85 mm
- net /IO2_5: track 12.2 -> 35.9 mm
- net /IO1_4: track 10.8 -> 32.1 mm
- net /IO2_1: track 16.9 -> 37.5 mm
- net /IO2_6: track 13.5 -> 33.7 mm
- net /SW5: track 24.6 -> 6.41 mm
- net /LED0: track 23.3 -> 6.74 mm
- net /LED3: track 23.7 -> 7.34 mm
- net /IO1_3: track 6.74 -> 22.9 mm
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