File: timelapse/2019-07-03_07:08:37_fpga_hat.kicad_pcb (KiCad board)
At the start: 4 copper layers, 65 x 56.5 mm, 90 parts, among them J1 2x20, J2 AudioJack3, J3 Conn_02x06_Top_Bottom, J4 Conn_02x06_Top_Bottom, J5 Conn_02x06_Top_Bottom, J6 Conn_01x02, SW1 PTS815, SW2 PTS815, SW3 PTS815, SW4 PTS815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

Commit message: Continue BGA route-out. SRAM connected, start heading out toward LEDs and IO.
Connections:
- U1 pad A11: /IO0_6 -> /IO0_0
- U1 pad A7: /IO0_4 -> /IO1_2
- U1 pad B8: /IO1_2 -> /IO0_4
- U1 pad C8: /IO0_0 -> /IO0_6
- U1 pad J8: /GP27_SDIO_DAT3 -> /GP22_SDIO_CLK
- U1 pad K6: /GP22_SDIO_CLK -> /GP27_SDIO_DAT3
Routing:
- net /IO0_4: track 22.6 -> 16.5 mm
- net /IO0_0: track 20.6 -> 17.7 mm
- net /IO0_6: track 17.7 -> 16.7 mm
- net /GP27_SDIO_DAT3: track 9.88 -> 9.20 mm
- net /GP22_SDIO_CLK: track 9.20 -> 9.88 mm
