File: timelapse/2019-07-03_17:28:54_fpga_hat.kicad_pcb (KiCad board)
At the start: 4 copper layers, 65 x 56.5 mm, 90 parts, among them J1 2x20, J2 AudioJack3, J3 Conn_02x06_Top_Bottom, J4 Conn_02x06_Top_Bottom, J5 Conn_02x06_Top_Bottom, J6 Conn_01x02, SW1 PTS815, SW2 PTS815, SW3 PTS815, SW4 PTS815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

Commit message: Continue routing
Parts:
- moved TP4 0.50 mm to (150.0, 97.0)
- moved TP5 0.50 mm to (150.0, 95.0)
- moved C15 0.41 mm to (125.5, 110.0)
Connections:
- U1 pad E8: /IO2_4 -> /IO2_1
- U1 pad F10: /IO2_0 -> /IO2_6
- U1 pad F9: /IO2_1 -> /SW6
- U1 pad G10: /IO2_6 -> /LED5
- U1 pad G11: /IO2_2 -> /LED7
- U1 pad G8: /IO2_3 -> /IO2_0
- U1 pad G9: /IO2_7 -> /LED6
- U1 pad H10: /GP14_UART_TXD -> /SW4
- U1 pad H11: /LED7 -> /LED4
- U1 pad H7: /SW5 -> /IO2_4
- U1 pad H9: /SW7 -> /GP25_SDIO_DAT1
- U1 pad J11: /LED6 -> /IO2_7
- U1 pad J5: /LED4 -> /IO2_2
- U1 pad J7: /GP26_SDIO_DAT2 -> /IO2_3
- U1 pad J8: /GP23_SDIO_CMD -> /GP27_SDIO_DAT3
- U1 pad K11: /SW6 -> /SW5
- U1 pad K5: /SW4 -> /GP14_UART_TXD
- U1 pad K7: /GP25_SDIO_DAT1 -> /SW7
- U1 pad L5: /LED5 -> /GP26_SDIO_DAT2
- U1 pad L7: /GP24_SDIO_DAT0 -> /GP23_SDIO_CMD
- U1 pad L8: /GP27_SDIO_DAT3 -> /GP24_SDIO_DAT0
Routing:
- net /SW7: track 39.7 -> 2.04 mm
- net /SW5: track 37.0 -> 6.74 mm
- net /GP26_SDIO_DAT2: track 35.4 -> 10.5 mm
- net /SW4: track 33.0 -> 8.53 mm
- net /GP24_SDIO_DAT0: track 25.2 -> 4.18 mm
- net /GP23_SDIO_CMD: track 24.2 -> 7.81 mm
- net /LED4: track 22.8 -> 6.62 mm
- net /GP22_SDIO_CLK: track 21.7 -> 9.20 mm
- net /IO2_7: track 16.7 -> 6.14 mm
- net /LED5: track 20.7 -> 10.4 mm
- net /GP27_SDIO_DAT3: track 19.6 -> 9.88 mm
- net /GP25_SDIO_DAT1: track 0.00 -> 8.89 mm
- net /IO2_4: track 22.5 -> 13.8 mm
- net /IO2_1: track 15.0 -> 22.2 mm
- net /IO2_5: track 17.9 -> 12.2 mm
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