File: timelapse/2019-07-03_18:11:15_fpga_hat.kicad_pcb (KiCad board)
At the start: 4 copper layers, 65 x 56.5 mm, 90 parts, among them J1 2x20, J2 AudioJack3, J3 Conn_02x06_Top_Bottom, J4 Conn_02x06_Top_Bottom, J5 Conn_02x06_Top_Bottom, J6 Conn_01x02, SW1 PTS815, SW2 PTS815, SW3 PTS815, SW4 PTS815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

Commit message: Continue routing
Connections:
- U1 pad H9: /SW7 -> /GP25_SDIO_DAT1
- U1 pad J8: /GP23_SDIO_CMD -> /GP27_SDIO_DAT3
- U1 pad K7: /GP25_SDIO_DAT1 -> /SW7
- U1 pad L7: /GP24_SDIO_DAT0 -> /GP23_SDIO_CMD
- U1 pad L8: /GP27_SDIO_DAT3 -> /GP24_SDIO_DAT0
Routing:
- net /SW7: track 39.7 -> 2.04 mm
- net /GP24_SDIO_DAT0: track 25.2 -> 4.18 mm
- net /GP23_SDIO_CMD: track 24.2 -> 7.81 mm
- net /GP26_SDIO_DAT2: track 35.4 -> 25.4 mm
- net /GP27_SDIO_DAT3: track 19.6 -> 9.88 mm
- net /GP25_SDIO_DAT1: track 0.00 -> 8.89 mm
- net /LED5: track 20.7 -> 20.0 mm
- net /SW4: track 33.0 -> 33.7 mm
- net /GP22_SDIO_CLK: track 21.7 -> 21.1 mm
