File: timelapse/2019-07-03_18:30:05_fpga_hat.kicad_pcb (KiCad board)
At the start: 4 copper layers, 65 x 56.5 mm, 90 parts, among them J1 2x20, J2 AudioJack3, J3 Conn_02x06_Top_Bottom, J4 Conn_02x06_Top_Bottom, J5 Conn_02x06_Top_Bottom, J6 Conn_01x02, SW1 PTS815, SW2 PTS815, SW3 PTS815, SW4 PTS815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

Commit message: Continue routing
Connections:
- U1 pad J8: /GP23_SDIO_CMD -> /GP27_SDIO_DAT3
- U1 pad L8: /GP27_SDIO_DAT3 -> /GP23_SDIO_CMD
Routing:
- net /GP27_SDIO_DAT3: track 19.6 -> 24.2 mm
- net /GP23_SDIO_CMD: track 24.2 -> 19.6 mm
Changed lines of the file:
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@@
       (net 2 +1V2))
     (pad J8 smd circle (at 1.6 2.4 180) (size 0.3 0.3) (layers F.Cu F.Paste F.Mask)
-      (net 41 /GP23_SDIO_CMD))
+      (net 39 /GP27_SDIO_DAT3))
     (pad K8 smd circle (at 1.6 3.2 180) (size 0.3 0.3) (layers F.Cu F.Paste F.Mask)
       (net 31 /GP13_FPGA_CDONE))
     (pad L8 smd circle (at 1.6 4 180) (size 0.3 0.3) (layers F.Cu F.Paste F.Mask)
-      (net 39 /GP27_SDIO_DAT3))
+      (net 41 /GP23_SDIO_CMD))
     (pad A9 smd circle (at 2.4 -4 180) (size 0.3 0.3) (layers F.Cu F.Paste F.Mask)
       (net 61 /IO0_2))
@@
   (segment (start 153.485 89) (end 153.485 89.6475) (width 0.09) (layer F.Cu) (net 29))
   (segment (start 153.9375 90.1) (end 153.9375 91) (width 0.09) (layer F.Cu) (net 29))
-  (segment (start 131.4 102.323625) (end 124.739978 95.663603) (width 0.09) (layer F.Cu) (net 41))
-  (segment (start 124.739978 83.760022) (end 125.4 83.1) (width 0.09) (layer F.Cu) (net 41))
-  (segment (start 124.739978 95.663603) (end 124.739978 83.760022) (width 0.09) (layer F.Cu) (net 41))
-  (segment (start 131.4 103.6) (end 131.4 102.323625) (width 0.09) (layer F.Cu) (net 41))
-  (segment (start 130.9 104.1) (end 131.4 103.6) (width 0.09) (layer F.Cu) (net 41))
+  (segment (start 131.4 102.323625) (end 124.739978 95.663603) (width 0.09) (layer F.Cu) (net 39))
+  (segment (start 124.739978 83.760022) (end 125.4 83.1) (width 0.09) (layer F.Cu) (net 39))
+  (segment (start 124.739978 95.663603) (end 124.739978 83.760022) (width 0.09) (layer F.Cu) (net 39))
+  (segment (start 131.4 103.6) (end 131.4 102.323625) (width 0.09) (layer F.Cu) (net 39))
+  (segment (start 130.9 104.1) (end 131.4 103.6) (width 0.09) (layer F.Cu) (net 39))
   (segment (start 132.180011 101.980011) (end 125.480011 95.280011) (width 0.09) (layer F.Cu) (net 40))
   (segment (start 125.480011 86.67207) (end 126.15 86.002081) (width 0.09) (layer F.Cu) (net 40))
@@
   (segment (start 124.919989 84.080011) (end 125.6 83.4) (width 0.09) (layer F.Cu) (net 42))
   (segment (start 125.6 83.4) (end 128.6 83.4) (width 0.09) (layer F.Cu) (net 42))
-  (segment (start 124.4 95.869052) (end 124.4 86.3) (width 0.09) (layer F.Cu) (net 39))
-  (segment (start 130.9 102.5) (end 130.9 102.369052) (width 0.09) (layer F.Cu) (net 39))
-  (segment (start 124.4 86.3) (end 123.9 85.8) (width 0.09) (layer F.Cu) (net 39))
-  (segment (start 130.9 102.369052) (end 124.4 95.869052) (width 0.09) (layer F.Cu) (net 39))
+  (segment (start 124.4 95.869052) (end 124.4 86.3) (width 0.09) (layer F.Cu) (net 41))
+  (segment (start 130.9 102.5) (end 130.9 102.369052) (width 0.09) (layer F.Cu) (net 41))
+  (segment (start 124.4 86.3) (end 123.9 85.8) (width 0.09) (layer F.Cu) (net 41))
+  (segment (start 130.9 102.369052) (end 124.4 95.869052) (width 0.09) (layer F.Cu) (net 41))
   (segment (start 132.1 103.7) (end 132.521802 103.7) (width 0.09) (layer F.Cu) (net 56))
   (segment (start 132.81999 103.401812) (end 132.81999 101.28001) (width 0.09) (layer F.Cu) (net 56))
