File: timelapse/2019-07-06_11:05:02_fpga_hat.kicad_pcb (KiCad board)
At the start: 4 copper layers, 65 x 56.5 mm, 91 parts, among them J1 2x20, J2 AudioJack3, J3 Conn_02x06_Top_Bottom, J4 Conn_02x06_Top_Bottom, J5 Conn_02x06_Top_Bottom, J6 Conn_01x02, SW1 PTS815, SW2 PTS815, SW3 PTS815, SW4 PTS815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

Commit message: Routed 100%
Parts:
- moved C24 0.46 mm to (109.5, 121.0)
- moved C13 0.30 mm to (115.5, 94.0)
- moved C23 0.26 mm to (132.0, 121.0)
- moved C25 0.20 mm to (120.5, 103.0)
- moved C19 0.12 mm to (159.0, 128.0)
- moved R7 0.10 mm to (162.0, 128.0)
- moved R9 0.10 mm to (160.5, 128.0)
Routing:
- net +3V3: track 46.8 -> 20.0 mm, vias 15 -> 11
- net /GP10_SPI_MOSI: track 28.9 -> 10.4 mm, vias 1 -> 0
- net Net-(C19-Pad1): track 14.5 -> 0.00 mm
- net Net-(C18-Pad1): track 9.45 -> 0.00 mm
- net +3.3VDAC: track 9.09 -> 0.00 mm, vias 1 -> 0
- net +5V: track 12.3 -> 5.96 mm, vias 3 -> 1
- net +1V2: track 18.2 -> 13.9 mm, vias 7 -> 6
- net Net-(C20-Pad1): track 4.12 -> 0.00 mm
- net Net-(C21-Pad1): track 3.47 -> 0.00 mm
- net Net-(R7-Pad2): track 2.89 -> 0.00 mm, vias 1 -> 0
- net Net-(R6-Pad2): track 2.88 -> 0.00 mm, vias 1 -> 0
- net Net-(C2-Pad1): track 4.35 -> 2.94 mm
- net GND: vias 67 -> 43
- net /GP13_FPGA_CDONE: vias 2 -> 4
- removed copper zone on F.Cu, net +1V2
- removed copper zone on F.Cu, net +5V
- removed copper zone on F.Cu, net Net-(L1-Pad1)
