File: timelapse/2019-07-06_11:30:20_fpga_hat.kicad_pcb (KiCad board)
At the start: 4 copper layers, 65 x 56.5 mm, 91 parts, among them J1 2x20, J2 AudioJack3, J3 Conn_02x06_Top_Bottom, J4 Conn_02x06_Top_Bottom, J5 Conn_02x06_Top_Bottom, J6 Conn_01x02, SW1 PTS815, SW2 PTS815, SW3 PTS815, SW4 PTS815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

Commit message: Routed 100%
Parts:
- moved C24 0.46 mm to (109.5, 121.0)
- moved C13 0.30 mm to (115.5, 94.0)
- moved C23 0.26 mm to (132.0, 121.0)
- moved C25 0.20 mm to (120.5, 103.0)
Routing:
- net /GP10_SPI_MOSI: track 28.9 -> 10.4 mm, vias 1 -> 0
- net +3V3: track 46.8 -> 33.3 mm, vias 15 -> 12
- net +1V2: track 18.2 -> 13.9 mm, vias 7 -> 6
- net Net-(C2-Pad1): track 4.35 -> 2.94 mm
- net +5V: track 12.3 -> 12.8 mm, vias 3 -> 2
- net GND: vias 67 -> 63
- net /GP13_FPGA_CDONE: vias 2 -> 3
- removed copper zone on F.Cu, net +1V2
- removed copper zone on F.Cu, net +5V
- removed copper zone on F.Cu, net Net-(L1-Pad1)
