File: timelapse/2019-07-06_11:52:16_fpga_hat.kicad_pcb (KiCad board)
At the start: 4 copper layers, 65 x 56.5 mm, 91 parts, among them J1 2x20, J2 AudioJack3, J3 Conn_02x06_Top_Bottom, J4 Conn_02x06_Top_Bottom, J5 Conn_02x06_Top_Bottom, J6 Conn_01x02, SW1 PTS815, SW2 PTS815, SW3 PTS815, SW4 PTS815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

Commit message: Routed 100%
Parts:
- moved C13 0.30 mm to (115.5, 94.0)
Routing:
- net +1V2: track 18.2 -> 13.9 mm, vias 7 -> 6
- net +5V: track 12.3 -> 12.8 mm, vias 3 -> 2
- net GND: vias 67 -> 63
- net /GP13_FPGA_CDONE: vias 2 -> 3
- removed copper zone on F.Cu, net +1V2
- removed copper zone on F.Cu, net +5V
- removed copper zone on F.Cu, net Net-(L1-Pad1)
Changed lines of the file:
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@@
     (thickness 1.6)
     (drawings 20)
-    (tracks 1220)
+    (tracks 1216)
     (zones 0)
     (modules 91)
@@
   )
   (setup
-    (last_trace_width 0.15)
+    (last_trace_width 0.5)
     (user_trace_width 0.15)
     (user_trace_width 0.25)
@@
   )
   (module Capacitor_SMD:C_0402_1005Metric (layer F.Cu)
-    (at 115.8 94 270)
+    (at 115.5 94 270)
     (descr "Capacitor SMD 0402 (1005 Metric), square (rectangular) end terminal, IPC_7351 nominal, (Body size source: http://www.tortai-tech.com/upload/download/2011102023233369053.pdf), generated with kicad-footprint-generator")
     (tags capacitor)
@@
   (segment (start 128.9 107.615) (end 129.615 107.615) (width 0.5) (layer B.Cu) (net 1))
   (via (at 119.6 96.5) (size 0.45) (drill 0.2) (layers F.Cu B.Cu) (net 1))
+  (segment (start 118.7875 96.5) (end 119.6 96.5) (width 0.5) (layer F.Cu) (net 1))
   (via (at 119.8 95.9) (size 0.45) (drill 0.2) (layers F.Cu B.Cu) (net 1))
+  (segment (start 119.7125 95) (end 119.7125 95.8125) (width 0.5) (layer F.Cu) (net 1))
+  (segment (start 119.7125 95.8125) (end 119.8 95.9) (width 0.5) (layer F.Cu) (net 1))
   (segment (start 117.25 94.25) (end 117.5 94) (width 0.25) (layer F.Cu) (net 1))
   (segment (start 117.25 95) (end 117.25 94.25) (width 0.25) (layer F.Cu) (net 1))
@@
   (via (at 130.5 104.5) (size 0.45) (drill 0.2) (layers F.Cu B.Cu) (net 2))
   (segment (start 130.9 104.9) (end 130.5 104.5) (width 0.25) (layer F.Cu) (net 2))
+  (segment (start 121.2875 94.2125) (end 121.2875 95) (width 0.5) (layer F.Cu) (net 2))
+  (segment (start 121.4375 94.0625) (end 121.2875 94.2125) (width 0.5) (layer F.Cu) (net 2))
+  (segment (start 121.4375 93) (end 121.4375 94.0625) (width 0.5) (layer F.Cu) (net 2))
+  (via (at 122.2 95) (size 0.6) (drill 0.3) (layers F.Cu B.Cu) (net 2))
+  (segment (start 121.2875 95) (end 122.2 95) (width 0.5) (layer F.Cu) (net 2))
   (via (at 121.3 96) (size 0.6) (drill 0.3) (layers F.Cu B.Cu) (net 2))
+  (segment (start 121.2875 95) (end 121.2875 95.9875) (width 0.5) (layer F.Cu) (net 2))
   (segment (start 121.2875 95.9875) (end 121.3 96) (width 0.5) (layer F.Cu) (net 2))
+  (segment (start 116.475 93) (end 116.75 93) (width 0.15) (layer F.Cu) (net 2))
+  (segment (start 115.5 93.515) (end 115.96 93.515) (width 0.15) (layer F.Cu) (net 2))
+  (segment (start 115.96 93.515) (end 116.475 93) (width 0.15) (layer F.Cu) (net 2))
   (segment (start 134.1 108.1) (end 133.7 107.7) (width 0.25) (layer F.Cu) (net 2))
   (via (at 133.7 107.7) (size 0.45) (drill 0.2) (layers F.Cu B.Cu) (net 2))
@@
   (segment (start 136.1 91) (end 136.1 91.7) (width 0.25) (layer F.Cu) (net 7))
   (segment (start 136.1 92.515) (end 136.1 91.7) (width 0.25) (layer F.Cu) (net 7))
+  (segment (start 117.75 95.9625) (end 117.2125 96.5) (width 0.25) (layer F.Cu) (net 8))
+  (segment (start 117.75 95) (end 117.75 95.9625) (width 0.25) (layer F.Cu) (net 8))
   (via (at 116.3 96.5) (size 0.45) (drill 0.2) (layers F.Cu B.Cu) (net 8))
   (segment (start 117.2125 96.5) (end 116.3 96.5) (width 0.5) (layer F.Cu) (net 8))
@@
   (segment (start 125.2125 127) (end 125.2125 128.10625) (width 0.5) (layer F.Cu) (net 8))
   (segment (start 125.2125 128.10625) (end 126 128.89375) (width 0.5) (layer F.Cu) (net 8))
+  (segment (start 116.5 95) (end 116.75 95) (width 0.15) (layer F.Cu) (net 9))
+  (segment (start 115.5 94.485) (end 115.985 94.485) (width 0.15) (layer F.Cu) (net 9))
+  (segment (start 115.985 94.485) (end 116.5 95) (width 0.15) (layer F.Cu) (net 9))
   (segment (start 153.9 118.9625) (end 153.9375 119) (width 0.09) (layer F.Cu) (net 15))
   (segment (start 153.9 118) (end 153.9 118.9625) (width 0.09) (layer F.Cu) (net 15))
@@
   (via (at 130.2 90.2) (size 0.45) (drill 0.2) (layers F.Cu B.Cu) (net 1) (status 40000))
   (via (at 130.5 87.8) (size 0.45) (drill 0.2) (layers F.Cu B.Cu) (net 1))
-  (segment (start 118.25 94.1) (end 118.25 95) (width 0.15) (layer F.Cu) (net 1))
-  (segment (start 117.5 94) (end 118.15 94) (width 0.15) (layer F.Cu) (net 1))
-  (segment (start 118.15 94) (end 118.25 94.1) (width 0.15) (layer F.Cu) (net 1))
-  (via (at 161.2 127.05) (size 0.45) (drill 0.2) (layers F.Cu B.Cu) (net 1))
-  (via (at 156.3 125.35) (size 0.45) (drill 0.2) (layers F.Cu B.Cu) (net 1))
-  (via (at 157.65 124.2) (size 0.45) (drill 0.2) (layers F.Cu B.Cu) (net 1))
-  (via (at 161.15 124.8) (size 0.45) (drill 0.2) (layers F.Cu B.Cu) (net 1))
-  (via (at 122.2 95) (size 0.6) (drill 0.3) (layers F.Cu B.Cu) (net 2))
-  (via (at 115.8 92.75) (size 0.45) (drill 0.2) (layers F.Cu B.Cu) (net 2))
-  (segment (start 122.2 95) (end 118.05 95) (width 0.15) (layer In2.Cu) (net 2))
-  (segment (start 118.05 95) (end 115.8 92.75) (width 0.15) (layer In2.Cu) (net 2))
-  (segment (start 116.75 92.55) (end 116.75 93) (width 0.15) (layer F.Cu) (net 2))
-  (segment (start 116.6 92.4) (end 116.75 92.55) (width 0.15) (layer F.Cu) (net 2))
-  (segment (start 115.8 92.75) (end 116.15 92.4) (width 0.15) (layer F.Cu) (net 2))
-  (segment (start 116.15 92.4) (end 116.6 92.4) (width 0.15) (layer F.Cu) (net 2))
-  (segment (start 115.8 92.75) (end 115.8 93.515) (width 0.15) (layer F.Cu) (net 2))
   (segment (start 131.3 103.125) (end 131.325 103.1) (width 0.5) (layer B.Cu) (net 4))
   (segment (start 131.3 104.5) (end 131.3 103.125) (width 0.5) (layer B.Cu) (net 4))
@@
   (segment (start 160.95 123.93) (end 160.93 123.95) (width 0.5) (layer F.Cu) (net 8))
   (segment (start 160.95 122.07) (end 160.95 123.93) (width 0.5) (layer F.Cu) (net 8))
-  (via (at 117.2 92.15) (size 0.45) (drill 0.2) (layers F.Cu B.Cu) (net 8))
-  (segment (start 117.45 92.15) (end 117.2 92.15) (width 0.15) (layer F.Cu) (net 8))
-  (segment (start 117.75 93) (end 117.75 92.45) (width 0.15) (layer F.Cu) (net 8))
-  (segment (start 117.75 92.45) (end 117.45 92.15) (width 0.15) (layer F.Cu) (net 8))
-  (segment (start 115.8 94.485) (end 116.315 95) (width 0.15) (layer F.Cu) (net 9))
-  (segment (start 116.315 95) (end 116.75 95) (width 0.15) (layer F.Cu) (net 9))
   (segment (start 162 125.5) (end 160.5 125.5) (width 0.15) (layer B.Cu) (net 10))
   (segment (start 160.08 125.5) (end 159 125.5) (width 0.15) (layer B.Cu) (net 10))
@@
   (segment (start 131.910898 98.879956) (end 143.920042 98.879956) (width 0.09) (layer B.Cu) (net 30))
   (segment (start 143.920042 98.879956) (end 150.275001 92.524997) (width 0.09) (layer B.Cu) (net 30))
+  (via (at 132.1 100.4) (size 0.45) (drill 0.2) (layers F.Cu B.Cu) (net 31) (status 40000))
   (segment (start 143.161426 98.438574) (end 148.2 93.4) (width 0.09) (layer B.Cu) (net 31))
   (segment (start 131.588574 98.438574) (end 143.161426 98.438574) (width 0.09) (layer B.Cu) (net 31))
@@
     (polygon
       (pts
-        (xy 112 77.5) (xy 112 83.5) (xy 107 83.5) (xy 107 86) (xy 112.25 91.25)
-        (xy 116.8 91.25) (xy 117.9 92.35) (xy 117.9 97.1) (xy 112.5 102.5) (xy 112.5 115.5)
-        (xy 106.5 121.5) (xy 106.5 128) (xy 125 128) (xy 152 128) (xy 160.5 119.5)
-        (xy 169.5 119.5) (xy 169.5 139) (xy 100 139) (xy 100 77.5) (xy 102 77.5)
+        (xy 112 77.5) (xy 112 83.5) (xy 107 83.5) (xy 107 86) (xy 117.5 96.5)
+        (xy 117.5 97.5) (xy 112.5 102.5) (xy 112.5 115.5) (xy 106.5 121.5) (xy 106.5 128)
+        (xy 125 128) (xy 152 128) (xy 160.5 119.5) (xy 169.5 119.5) (xy 169.5 139)
+        (xy 100 139) (xy 100 77.5) (xy 102 77.5)
       )
     )
@@
       )
     )
-  )
-  (zone (net 2) (net_name +1V2) (layer F.Cu) (hatch edge 0.508)
-    (priority 2)
-    (connect_pads yes (clearance 0.1))
-    (min_thickness 0.1)
-    (fill yes (arc_segments 32) (thermal_gap 0.508) (thermal_bridge_width 0.508))
-    (polygon
-      (pts
-        (xy 120.8 91.95) (xy 122.35 91.95) (xy 123.1 92.7) (xy 123.1 96.45) (xy 122.35 97.2)
-        (xy 121.15 97.2) (xy 120.8 96.85)
-      )
-    )
-  )
-  (zone (net 1) (net_name GND) (layer F.Cu) (hatch edge 0.508)
-    (priority 2)
-    (connect_pads yes (clearance 0.1))
-    (min_thickness 0.1)
-    (fill yes (arc_segments 32) (thermal_gap 0.508) (thermal_bridge_width 0.508))
-    (polygon
-      (pts
-        (xy 118.1 94.55) (xy 118.1 94.4) (xy 117.95 94.25) (xy 117.95 93.7) (xy 118.45 94.2)
-        (xy 120.4 94.2) (xy 120.4 97.2) (xy 118.1 97.2)
-      )
-    )
-  )
-  (zone (net 84) (net_name "Net-(L1-Pad1)") (layer F.Cu) (hatch edge 0.508)
-    (priority 2)
-    (connect_pads yes (clearance 0.1))
-    (min_thickness 0.1)
-    (fill yes (arc_segments 32) (thermal_gap 0.508) (thermal_bridge_width 0.508))
-    (polygon
-      (pts
-        (xy 118.15 92.65) (xy 118.75 92.05) (xy 120.1 92.05) (xy 120.3 92.25) (xy 120.3 93.7)
-        (xy 120 94) (xy 118.85 94) (xy 118.15 93.3)
-      )
-    )
-  )
-  (zone (net 8) (net_name +5V) (layer F.Cu) (hatch edge 0.508)
-    (priority 2)
-    (connect_pads yes (clearance 0.1))
-    (min_thickness 0.1)
-    (fill yes (arc_segments 32) (thermal_gap 0.508) (thermal_bridge_width 0.508))
-    (polygon
-      (pts
-        (xy 117.6 94.65) (xy 117.9 94.65) (xy 117.9 96.8) (xy 117.5 97.2) (xy 116.5 97.2)
-        (xy 116 96.7) (xy 116 96.3) (xy 116.5 95.8) (xy 117.3 95.8) (xy 117.6 95.5)
-      )
-    )
