File: timelapse/2019-07-06_12:26:53_fpga_hat.kicad_pcb (KiCad board)
At the start: 4 copper layers, 65 x 56.5 mm, 91 parts, among them J1 2x20, J2 AudioJack3, J3 Conn_02x06_Top_Bottom, J4 Conn_02x06_Top_Bottom, J5 Conn_02x06_Top_Bottom, J6 Conn_01x02, SW1 PTS815, SW2 PTS815, SW3 PTS815, SW4 PTS815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

Commit message: Routed 100%
Routing:
- net GND: vias 67 -> 63
- net /GP13_FPGA_CDONE: vias 2 -> 3
Changed lines of the file:
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@@
     (thickness 1.6)
     (drawings 20)
-    (tracks 1220)
+    (tracks 1217)
     (zones 0)
     (modules 91)
@@
   (segment (start 117.5 94) (end 118.15 94) (width 0.15) (layer F.Cu) (net 1))
   (segment (start 118.15 94) (end 118.25 94.1) (width 0.15) (layer F.Cu) (net 1))
-  (via (at 161.2 127.05) (size 0.45) (drill 0.2) (layers F.Cu B.Cu) (net 1))
-  (via (at 156.3 125.35) (size 0.45) (drill 0.2) (layers F.Cu B.Cu) (net 1))
-  (via (at 157.65 124.2) (size 0.45) (drill 0.2) (layers F.Cu B.Cu) (net 1))
-  (via (at 161.15 124.8) (size 0.45) (drill 0.2) (layers F.Cu B.Cu) (net 1))
   (via (at 122.2 95) (size 0.6) (drill 0.3) (layers F.Cu B.Cu) (net 2))
   (via (at 115.8 92.75) (size 0.45) (drill 0.2) (layers F.Cu B.Cu) (net 2))
@@
   (segment (start 131.910898 98.879956) (end 143.920042 98.879956) (width 0.09) (layer B.Cu) (net 30))
   (segment (start 143.920042 98.879956) (end 150.275001 92.524997) (width 0.09) (layer B.Cu) (net 30))
+  (via (at 132.1 100.4) (size 0.45) (drill 0.2) (layers F.Cu B.Cu) (net 31) (status 40000))
   (segment (start 143.161426 98.438574) (end 148.2 93.4) (width 0.09) (layer B.Cu) (net 31))
   (segment (start 131.588574 98.438574) (end 143.161426 98.438574) (width 0.09) (layer B.Cu) (net 31))
