File: timelapse/2019-07-06_13:41:26_fpga_hat.kicad_pcb (KiCad board)
At the start: 4 copper layers, 65 x 56.5 mm, 92 parts, among them J1 2x20, J2 AudioJack3, J3 Conn_02x06_Top_Bottom, J4 Conn_02x06_Top_Bottom, J5 Conn_02x06_Top_Bottom, J6 Conn_01x02, SW1 PTS815, SW2 PTS815, SW3 PTS815, SW4 PTS815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

Commit message: Add pinout on silkscreen, move TP5
Parts:
- moved TP5 8.28 mm to (149.5, 95.0)
- moved C25 4.71 mm to (120.3, 103.0), turned to 270 degrees
- moved C24 4.71 mm to (109.1, 121.2), turned to 0 degrees
- moved C23 4.70 mm to (131.8, 121.2), turned to 0 degrees
- moved REF** 0.20 mm to (125.5, 114.5)
Routing:
- net /GP12_FPGA_~RST: track 47.3 -> 49.4 mm
Other:
- board text removed: "+5V"
- board text removed: "0"
- board text removed: "1"
- board text removed: "2"
- board text removed: "3"
- board text removed: "3V3"
- board text removed: "4"
- board text removed: "5"
- board text removed: "6"
- board text removed: "7"
- board text removed: "GND"
- board text removed: "IO Header 0"
- board text removed: "IO Header 1"
- board text removed: "IO Header 2"
